Commit message: created a hardware driver to test the actual robotic arm

File: base_station_ws/misbah_arm_temp/src/arm_moveit_config/config/rover_arm.ros2_control.xacro (robot description, xacro)
@@ -1,36 +1,125 @@
 <?xml version="1.0"?>
 <robot xmlns:xacro="http://www.ros.org/wiki/xacro">
-    <xacro:macro name="rover_arm_ros2_control" params="name initial_positions_file">
+    <xacro:macro name="rover_arm_ros2_control"
+                 params="name initial_positions_file use_mock_hardware:=^|true can_interface:=^|can0 base_joint_connected:=^|true">
         <xacro:property name="initial_positions" value="${xacro.load_yaml(initial_positions_file)['initial_positions']}"/>
-        <ros2_control name="${name}" type="system">
-            <hardware>
-                <!-- By default, set up controllers for simulation. This won't work on real hardware -->
-                <plugin>mock_components/GenericSystem</plugin>
-            </hardware>
-            <joint name="base_joint">
-                <command_interface name="position"/>
-                <command_interface name="velocity"/>
-                <state_interface name="position">
-                  <param name="initial_value">${initial_positions['base_joint']}</param>
-                </state_interface>
-                <state_interface name="velocity"/>
-            </joint>
-            <joint name="shoulder_joint">
-                <command_interface name="position"/>
-                <command_interface name="velocity"/>
-                <state_interface name="position">
-                  <param name="initial_value">${initial_positions['shoulder_joint']}</param>
-                </state_interface>
-                <state_interface name="velocity"/>
-            </joint>
-            <joint name="elbow_joint">
-                <command_interface name="position"/>
-                <command_interface name="velocity"/>
-                <state_interface name="position">
-                  <param name="initial_value">${initial_positions['elbow_joint']}</param>
-                </state_interface>
-                <state_interface name="velocity"/>
-            </joint>
-        </ros2_control>
+        <!-- ═══════════════════════════════════════════════════════════
+             Case 1: MOCK — all joints simulated in one block
+             (used by demo.launch.py and any use_mock_hardware:=true call)
+             ═══════════════════════════════════════════════════════════ -->
+        <xacro:if value="${use_mock_hardware}">
+            <ros2_control name="${name}" type="system">
+                <hardware>
+                    <plugin>mock_components/GenericSystem</plugin>
+                </hardware>
+                <joint name="base_joint">
+                    <command_interface name="position"/>
+                    <command_interface name="velocity"/>
+                    <state_interface name="position">
+                        <param name="initial_value">${initial_positions['base_joint']}</param>
+                    </state_interface>
+                    <state_interface name="velocity"/>
+                </joint>
+                <joint name="shoulder_joint">
+                    <command_interface name="position"/>
+                    <command_interface name="velocity"/>
+                    <state_interface name="position">
+                        <param name="initial_value">${initial_positions['shoulder_joint']}</param>
+                    </state_interface>
+                    <state_interface name="velocity"/>
+                </joint>
+                <joint name="elbow_joint">
+                    <command_interface name="position"/>
+                    <command_interface name="velocity"/>
+                    <state_interface name="position">
+                        <param name="initial_value">${initial_positions['elbow_joint']}</param>
+                    </state_interface>
+                    <state_interface name="velocity"/>
+                </joint>
+            </ros2_control>
+        </xacro:if>
+        <!-- ═══════════════════════════════════════════════════════════
+             Cases 2 & 3: REAL hardware
+             ═══════════════════════════════════════════════════════════ -->
+        <xacro:unless value="${use_mock_hardware}">
+            <!-- Case 2: all 3 motors physically connected → one CAN block -->
+            <xacro:if value="${base_joint_connected}">
+                <ros2_control name="${name}" type="system">
+                    <hardware>
+                        <plugin>my_robot_hardware/ArmHardwareInterface</plugin>
+                        <param name="can_interface">${can_interface}</param>
+                    </hardware>
+                    <joint name="base_joint">
+                        <command_interface name="position"/>
+                        <command_interface name="velocity"/>
+                        <state_interface name="position">
+                            <param name="initial_value">${initial_positions['base_joint']}</param>
+                        </state_interface>
+                        <state_interface name="velocity"/>
+                        <param name="can_id">1</param>
+                    </joint>
+                    <joint name="shoulder_joint">
+                        <command_interface name="position"/>
+                        <command_interface name="velocity"/>
+                        <state_interface name="position">
+                            <param name="initial_value">${initial_positions['shoulder_joint']}</param>
+                        </state_interface>
+                        <state_interface name="velocity"/>
+                        <param name="can_id">2</param>
+                    </joint>
+                    <joint name="elbow_joint">
+                        <command_interface name="position"/>
+                        <command_interface name="velocity"/>
+                        <state_interface name="position">
+                            <param name="initial_value">${initial_positions['elbow_joint']}</param>
+                        </state_interface>
+                        <state_interface name="velocity"/>
+                        <param name="can_id">3</param>
+                    </joint>
+                </ros2_control>
+            </xacro:if>
+            <!-- Case 3: base_joint NOT connected → mock base, real CAN for shoulder+elbow -->
+            <xacro:unless value="${base_joint_connected}">
+                <!-- base_joint: simulated (motor not physically present) -->
+                <ros2_control name="${name}_base_mock" type="system">
+                    <hardware>
+                        <plugin>mock_components/GenericSystem</plugin>
+                    </hardware>
+                    <joint name="base_joint">
+                        <command_interface name="position"/>
+                        <command_interface name="velocity"/>
+                        <state_interface name="position">
+                            <param name="initial_value">${initial_positions['base_joint']}</param>
+                        </state_interface>
+                        <state_interface name="velocity"/>
+                    </joint>
+                </ros2_control>
+                <!-- shoulder + elbow: real SocketCAN hardware -->
+                <ros2_control name="${name}" type="system">
+                    <hardware>
+                        <plugin>my_robot_hardware/ArmHardwareInterface</plugin>
+                        <param name="can_interface">${can_interface}</param>
+                    </hardware>
+                    <joint name="shoulder_joint">
+                        <command_interface name="position"/>
+                        <command_interface name="velocity"/>
+                        <state_interface name="position">
+                            <param name="initial_value">${initial_positions['shoulder_joint']}</param>
+                        </state_interface>
+                        <state_interface name="velocity"/>
+                        <param name="can_id">2</param>
+                    </joint>
+                    <joint name="elbow_joint">
+                        <command_interface name="position"/>
+                        <command_interface name="velocity"/>
+                        <state_interface name="position">
+                            <param name="initial_value">${initial_positions['elbow_joint']}</param>
+                        </state_interface>
+                        <state_interface name="velocity"/>
+                        <param name="can_id">3</param>
+                    </joint>
+                </ros2_control>
+            </xacro:unless>
+        </xacro:unless>
     </xacro:macro>
 </robot>

File: base_station_ws/misbah_arm_temp/src/arm_moveit_config/config/rover_arm.urdf.xacro (robot description, xacro)
@@ -2,8 +2,16 @@
 <robot xmlns:xacro="http://www.ros.org/wiki/xacro" name="rover_arm">
     <xacro:arg name="initial_positions_file" default="initial_positions.yaml" />
+    <xacro:arg name="use_mock_hardware"      default="true" />
+    <xacro:arg name="can_interface"          default="can0" />
+    <xacro:arg name="base_joint_connected"   default="true" />
     <!-- Import rover_arm urdf file -->
     <xacro:include filename="$(find arm_description)/urdf/arm.urdf" />
     <!-- Import control_xacro -->
     <xacro:include filename="rover_arm.ros2_control.xacro" />
-    <xacro:rover_arm_ros2_control name="FakeSystem" initial_positions_file="$(arg initial_positions_file)"/>
+    <xacro:rover_arm_ros2_control
+        name="RoverArmSystem"
+        initial_positions_file="$(arg initial_positions_file)"
+        use_mock_hardware="$(arg use_mock_hardware)"
+        can_interface="$(arg can_interface)"
+        base_joint_connected="$(arg base_joint_connected)" />
 </robot>
