Commit message: added ros2_control files for drive train

File: rpi_ws/src/rover_description/urdf/rover.urdf.xacro (robot description, xacro)
@@ -12,4 +12,6 @@
 -->
 <robot xmlns:xacro="http://www.ros.org/wiki/xacro" name="deakin_rover">
+  <!-- ros2_control mock toggle — set false for real hardware -->
+  <xacro:arg name="use_mock_hardware" default="true"/>
   <!-- ==================== PROPERTIES ==================== -->
   <!-- Chassis dimensions (meters) — HARDWARE UPGRADE: measure real rover -->
@@ -95,4 +97,49 @@
   <xacro:wheel name="right_mid_wheel"   x="${mid_x}"   y="${-wheel_separation/2}"/>
   <xacro:wheel name="right_rear_wheel"  x="${rear_x}"  y="${-wheel_separation/2}"/>
+  <!-- ==================== ROS2_CONTROL ==================== -->
+  <!--
+    Hardware interface for the 6 BLD-3055 drive motors.
+    Modbus slave IDs: 1-3 left side, 4-6 right side (right side physically reversed).
+    HARDWARE UPGRADE: set use_mock to false and verify serial_port via dmesg.
+  -->
+  <ros2_control name="rover_drive" type="system">
+    <hardware>
+      <plugin>rover_drive_hardware/RoverDriveHardware</plugin>
+      <param name="serial_port">/dev/ttyUSB0</param>   <!-- HARDWARE UPGRADE: verify with dmesg -->
+      <param name="baud_rate">9600</param>              <!-- HARDWARE UPGRADE: can increase to 115200 -->
+      <param name="max_rpm">3000</param>                <!-- BLD-3055 datasheet limit -->
+      <param name="use_mock">$(arg use_mock_hardware)</param>
+    </hardware>
+    <joint name="left_front_wheel_joint">
+      <command_interface name="velocity"/>
+      <state_interface name="velocity"/>
+      <state_interface name="position"/>
+    </joint>
+    <joint name="left_mid_wheel_joint">
+      <command_interface name="velocity"/>
+      <state_interface name="velocity"/>
+      <state_interface name="position"/>
+    </joint>
+    <joint name="left_rear_wheel_joint">
+      <command_interface name="velocity"/>
+      <state_interface name="velocity"/>
+      <state_interface name="position"/>
+    </joint>
+    <joint name="right_front_wheel_joint">
+      <command_interface name="velocity"/>
+      <state_interface name="velocity"/>
+      <state_interface name="position"/>
+    </joint>
+    <joint name="right_mid_wheel_joint">
+      <command_interface name="velocity"/>
+      <state_interface name="velocity"/>
+      <state_interface name="position"/>
+    </joint>
+    <joint name="right_rear_wheel_joint">
+      <command_interface name="velocity"/>
+      <state_interface name="velocity"/>
+      <state_interface name="position"/>
+    </joint>
+  </ros2_control>
   <!-- ==================== ARM ==================== -->
   <!-- Base plate (flat cylinder, matches arm.urdf base_link) -->
